Commit message: This is the initial commit for indigo-devel. - sphero_driver.py was modified to try and reduce the connection errors, with a bad SOF - sphero_gui is a node that will connect the sphero and a hokuyo lidar to a RVIZ display this is still in progress - sphero_node/nodes/sphero.py has been modified to remove the queue_size warnings on startup and now normalizes the quaternion values on each packet received.

File: sphero_description/urdf/sphero.urdf (robot description, URDF)
Before this commit: robot sphero, 1 links, 0 joints
Links:
- added link base_footprint
- added link imu_link
Joints:
- added joint base_footprint_joint: type fixed, parent base_footprint, child base_link, origin xyz=0 0 0.0381 rpy=0 0 0
- added joint imu_joint: type fixed, parent base_footprint, child imu_link, origin xyz=0 0 0.0381 rpy=0 0 0
